Commit message: Fixed rename for master_thesis

File: gazebo/turtlebot3_description/urdf/turtlebot3_thesis.urdf.xacro (robot description, xacro)
@@ -1,6 +1,6 @@
 <?xml version="1.0" ?>
 <robot name="turtlebot3_thesis" xmlns:xacro="http://ros.org/wiki/xacro">
-  <xacro:include filename="$(find turtlebot3_description)/urdf/common_properties.xacro"/>
-  <xacro:include filename="$(find turtlebot3_description)/urdf/turtlebot3_thesis.gazebo.xacro"/>
+  <xacro:include filename="$(find master_thesis)/gazebo/turtlebot3_description/urdf/common_properties.xacro"/>
+  <xacro:include filename="$(find master_thesis)/gazebo/turtlebot3_description/urdf/turtlebot3_thesis.gazebo.xacro"/>
   <xacro:property name="r200_cam_rgb_px" value="0.000"/>
   <xacro:property name="r200_cam_rgb_py" value="0.00"/>
@@ -17,5 +17,5 @@
       <origin xyz="-0.064 0 0.0" rpy="0 0 0"/>
       <geometry>
-        <mesh filename="package://turtlebot3_description/meshes/bases/tb3_base.stl" scale="1.0 1.0 1.0"/>
+        <mesh filename="package://master_thesis/gazebo/turtlebot3_description/meshes/bases/tb3_base.stl" scale="1.0 1.0 1.0"/>
       </geometry>
       <material name="grey"/>
@@ -45,5 +45,5 @@
       <origin xyz="0 0 0" rpy="1.57 0 0"/>
       <geometry>
-        <mesh filename="package://turtlebot3_description/meshes/wheels/left_tire.stl" scale="0.001 0.001 0.001"/>
+        <mesh filename="package://master_thesis/gazebo/turtlebot3_description/meshes/wheels/left_tire.stl" scale="0.001 0.001 0.001"/>
       </geometry>
       <material name="dark"/>
@@ -73,5 +73,5 @@
       <origin xyz="0 0 0" rpy="1.57 0 0"/>
       <geometry>
-        <mesh filename="package://turtlebot3_description/meshes/wheels/right_tire.stl" scale="0.001 0.001 0.001"/>
+        <mesh filename="package://master_thesis/gazebo/turtlebot3_description/meshes/wheels/right_tire.stl" scale="0.001 0.001 0.001"/>
       </geometry>
       <material name="dark"/>
@@ -146,5 +146,5 @@
      <origin xyz="0 0 0" rpy="0 0 0"/>
       <geometry>
-       <mesh filename="package://turtlebot3_description/meshes/bases/sensor_base.stl" />
+       <mesh filename="package://master_thesis/gazebo/turtlebot3_description/meshes/bases/sensor_base.stl" />
       </geometry>
     </visual>
@@ -165,5 +165,5 @@
       <origin xyz="0 0 0" rpy="0 0 0"/>
       <geometry>
-        <mesh filename="package://turtlebot3_description/meshes/sensors/lds.stl" scale="0.001 0.001 0.001"/>
+        <mesh filename="package://master_thesis/gazebo/turtlebot3_description/meshes/sensors/lds.stl" scale="0.001 0.001 0.001"/>
       </geometry>
       <material name="dark"/>
@@ -185,5 +185,5 @@
      <origin xyz="0 0 0" rpy="1.57 0 1.57"/>
       <geometry>
-       <mesh filename="package://turtlebot3_description/meshes/sensors/hc-sr04.stl" />
+       <mesh filename="package://master_thesis/gazebo/turtlebot3_description/meshes/sensors/hc-sr04.stl" />
       </geometry>
       <material name="blue"/>
